File: Kicad/LEDHat/LEDHat.kicad_pcb (KiCad board)
At the start: 2 copper layers, 66 x 56 mm, 27 parts, among them J1 Conn_02x20_Odd_Even, J2 Conn_01x02_Male, Q1 2N7002E, Q2 2N7002E, Q3 2N7002E, Q4 2N7002E

Commit message: added PCB Design
Parts:
- moved J2 1.12 mm to (61.4, 73.3)
Routing:
- net +12V: track 92.0 -> 93.7 mm, vias 3 -> 4
- net GND: track 46.8 -> 46.7 mm, vias 23 -> 25
- net Net-(J1-Pad35): vias 2 -> 1
Other:
- board size 66 x 56 mm -> 65 x 56 mm
Changed lines of the file:
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@@
   )
   (footprint "Connector_PinHeader_2.54mm:PinHeader_1x02_P2.54mm_Horizontal" (layer "F.Cu")
-    (at 61.875 74.275 180)
+    (at 61.375 73.275 180)
     (descr "Through hole angled pin header, 1x02, 2.54mm pitch, 6mm pin length, single row")
     (tags "Through hole angled pin header THT 1x02 2.54mm single row")
@@
     )
   )
-  (gr_rect (start 49.5 60) (end 115.5 116) (layer "Edge.Cuts") (width 0.1) (fill none))
+  (gr_arc (start 53.5 116) (mid 51.025126 114.974874) (end 50 112.5) (layer "Edge.Cuts") (width 0.1))
+  (gr_arc (start 50 63.5) (mid 51.025126 61.025126) (end 53.5 60) (layer "Edge.Cuts") (width 0.1))
   (gr_circle (center 81.5 94) (end 81.5 82) (layer "Edge.Cuts") (width 0.1) (fill none))
+  (gr_line (start 111.5 116) (end 53.5 116) (layer "Edge.Cuts") (width 0.1))
+  (gr_arc (start 111.5 60) (mid 113.974874 61.025126) (end 115 63.5) (layer "Edge.Cuts") (width 0.1))
+  (gr_arc (start 115 112.5) (mid 113.974874 114.974874) (end 111.5 116) (layer "Edge.Cuts") (width 0.1))
+  (gr_line (start 53.5 60) (end 111.5 60) (layer "Edge.Cuts") (width 0.1))
+  (gr_line (start 50 112.5) (end 50 63.5) (layer "Edge.Cuts") (width 0.1))
+  (gr_line (start 115 63.5) (end 115 112.5) (layer "Edge.Cuts") (width 0.1))
   (gr_line (start 65.5 94) (end 97.5 94) (layer "User.1") (width 0.15))
   (gr_circle (center 81.5 94) (end 81.5 82) (layer "User.1") (width 0.15) (fill none))
@@
   (gr_rect (start 65.5 110) (end 97.5 78) (layer "User.1") (width 0.15) (fill none))
   (gr_line (start 76.5 78.5) (end 86.5 109) (layer "User.1") (width 0.15))
-  (gr_text "12V" (at 55 76.5 270) (layer "F.SilkS")
+  (gr_text "12V" (at 53.5 73.5 270) (layer "B.SilkS")
+    (effects (font (size 1 1) (thickness 0.15)) (justify mirror))
+  )
+  (gr_text "GND" (at 53.5 70.5 270) (layer "B.SilkS")
+    (effects (font (size 1 1) (thickness 0.15)) (justify mirror))
+  )
+  (gr_text "12V" (at 53.5 73.5 270) (layer "F.SilkS")
     (effects (font (size 1 1) (thickness 0.15)))
   )
@@
     (effects (font (size 1 1) (thickness 0.15)))
   )
-  (gr_text "GND\n" (at 55 69.5 270) (layer "F.SilkS")
+  (gr_text "GND\n" (at 53.5 70.5 270) (layer "F.SilkS")
     (effects (font (size 1 1) (thickness 0.15)))
   )
@@
   (segment (start 111.264 99.084) (end 102.5625 90.3825) (width 0.6) (layer "F.Cu") (net 14))
   (segment (start 102.5625 90.3825) (end 102.5625 73.95) (width 0.6) (layer "F.Cu") (net 14))
-  (segment (start 66.7775 71.735) (end 61.875 71.735) (width 0.6) (layer "F.Cu") (net 22))
-  (segment (start 68.0625 70.45) (end 66.7775 71.735) (width 0.6) (layer "F.Cu") (net 22))
+  (segment (start 59.765 70.735) (end 61.375 70.735) (width 0.6) (layer "F.Cu") (net 22))
+  (segment (start 61.375 70.735) (end 67.7775 70.735) (width 0.6) (layer "F.Cu") (net 22))
+  (segment (start 62.615 70.735) (end 61.375 70.735) (width 0.5) (layer "F.Cu") (net 22))
+  (segment (start 52 78.5) (end 59.765 70.735) (width 0.6) (layer "F.Cu") (net 22))
   (segment (start 52 96.19) (end 52 78.5) (width 0.6) (layer "F.Cu") (net 22))
-  (segment (start 58.765 71.735) (end 61.875 71.735) (width 0.6) (layer "F.Cu") (net 22))
-  (segment (start 61.875 71.735) (end 68.56 65.05) (width 0.6) (layer "F.Cu") (net 22))
-  (segment (start 68.56 65.05) (end 68.56 64.79) (width 0.6) (layer "F.Cu") (net 22))
-  (segment (start 52 78.5) (end 58.765 71.735) (width 0.6) (layer "F.Cu") (net 22))
+  (segment (start 68.56 64.79) (end 62.615 70.735) (width 0.5) (layer "F.Cu") (net 22))
+  (segment (start 67.7775 70.735) (end 68.0625 70.45) (width 0.6) (layer "F.Cu") (net 22))
   (via (at 61 79) (size 0.8) (drill 0.4) (layers "F.Cu" "B.Cu") (free) (net 22))
   (via (at 100.5 68) (size 0.8) (drill 0.4) (layers "F.Cu" "B.Cu") (free) (net 22))
@@
   (via (at 58.5 92.5) (size 0.8) (drill 0.4) (layers "F.Cu" "B.Cu") (free) (net 22))
   (via (at 60 103) (size 0.8) (drill 0.4) (layers "F.Cu" "B.Cu") (free) (net 22))
-  (via (at 59.5 68) (size 0.8) (drill 0.4) (layers "F.Cu" "B.Cu") (free) (net 22))
+  (via (at 92.5 75.5) (size 0.8) (drill 0.4) (layers "F.Cu" "B.Cu") (free) (net 22))
+  (via (at 110 68) (size 0.8) (drill 0.4) (layers "F.Cu" "B.Cu") (free) (net 22))
   (via (at 56.5 95.5) (size 0.8) (drill 0.4) (layers "F.Cu" "B.Cu") (free) (net 22))
   (via (at 81 112) (size 0.8) (drill 0.4) (layers "F.Cu" "B.Cu") (free) (net 22))
@@
   (via (at 102 97.5) (size 0.8) (drill 0.4) (layers "F.Cu" "B.Cu") (free) (net 22))
   (via (at 60 83.5) (size 0.8) (drill 0.4) (layers "F.Cu" "B.Cu") (free) (net 22))
-  (via (at 56 68) (size 0.8) (drill 0.4) (layers "F.Cu" "B.Cu") (free) (net 22))
+  (via (at 56 67) (size 0.8) (drill 0.4) (layers "F.Cu" "B.Cu") (free) (net 22))
   (via (at 106.5 97.5) (size 0.8) (drill 0.4) (layers "F.Cu" "B.Cu") (free) (net 22))
   (via (at 57.5 103) (size 0.8) (drill 0.4) (layers "F.Cu" "B.Cu") (free) (net 22))
+  (via (at 71 76) (size 0.8) (drill 0.4) (layers "F.Cu" "B.Cu") (free) (net 22))
   (via (at 59.5 106.5) (size 0.8) (drill 0.4) (layers "F.Cu" "B.Cu") (free) (net 22))
   (via (at 78.5 71) (size 0.8) (drill 0.4) (layers "F.Cu" "B.Cu") (free) (net 22))
@@
   (segment (start 111 83.5625) (end 109.4375 82) (width 0.6) (layer "F.Cu") (net 53))
   (segment (start 53.5 79.5) (end 56.65 79.5) (width 0.6) (layer "F.Cu") (net 53))
+  (segment (start 83.775 73.275) (end 84 73.5) (width 0.6) (layer "F.Cu") (net 53))
   (segment (start 109.4375 78) (end 109.4375 82) (width 0.6) (layer "F.Cu") (net 53))
-  (segment (start 56.65 79.5) (end 61.875 74.275) (width 0.6) (layer "F.Cu") (net 53))
+  (segment (start 56.65 79.5) (end 61.375 74.775) (width 0.6) (layer "F.Cu") (net 53))
+  (segment (start 61.375 73.275) (end 83.775 73.275) (width 0.6) (layer "F.Cu") (net 53))
   (segment (start 114 74.5) (end 114 73.5625) (width 0.6) (layer "F.Cu") (net 53))
   (segment (start 104.4375 73) (end 109.21875 77.78125) (width 0.6) (layer "F.Cu") (net 53))
+  (segment (start 61.375 74.775) (end 61.375 73.275) (width 0.6) (layer "F.Cu") (net 53))
   (segment (start 114 73.5625) (end 112.4375 72) (width 0.6) (layer "F.Cu") (net 53))
   (segment (start 109.21875 77.78125) (end 111 76) (width 0.6) (layer "F.Cu") (net 53))
@@
   (segment (start 109.21875 77.78125) (end 109.4375 78) (width 0.6) (layer "F.Cu") (net 53))
   (via (at 114 74.5) (size 0.8) (drill 0.4) (layers "F.Cu" "B.Cu") (net 53))
+  (via (at 84 73.5) (size 0.8) (drill 0.4) (layers "F.Cu" "B.Cu") (net 53))
   (via (at 111 85.5) (size 0.8) (drill 0.4) (layers "F.Cu" "B.Cu") (net 53))
   (via (at 111 76) (size 0.8) (drill 0.4) (layers "F.Cu" "B.Cu") (net 53))
   (segment (start 112.5 76) (end 114 74.5) (width 0.6) (layer "B.Cu") (net 53))
-  (segment (start 61.875 74.275) (end 98.225 74.275) (width 0.6) (layer "B.Cu") (net 53))
   (segment (start 100.5 76.55) (end 100.5 82) (width 0.6) (layer "B.Cu") (net 53))
   (segment (start 104 85.5) (end 111 85.5) (width 0.6) (layer "B.Cu") (net 53))
-  (segment (start 98.225 74.275) (end 100.5 76.55) (width 0.6) (layer "B.Cu") (net 53))
   (segment (start 100.5 82) (end 104 85.5) (width 0.6) (layer "B.Cu") (net 53))
   (segment (start 111 76) (end 112.5 76) (width 0.6) (layer "B.Cu") (net 53))
-  (segment (start 110.5625 71.05) (end 108.05 71.05) (width 0.6) (layer "F.Cu") (net 55))
-  (segment (start 108.05 71.05) (end 107 70) (width 0.6) (layer "F.Cu") (net 55))
-  (via (at 107 70) (size 0.8) (drill 0.4) (layers "F.Cu" "B.Cu") (net 55))
-  (via (at 101.58 64.79) (size 0.8) (drill 0.4) (layers "F.Cu" "B.Cu") (net 55))
-  (segment (start 101.58 64.79) (end 106.79 70) (width 0.6) (layer "B.Cu") (net 55))
-  (segment (start 106.79 70) (end 107 70) (width 0.6) (layer "B.Cu") (net 55))
+  (segment (start 97.45 73.5) (end 100.5 76.55) (width 0.6) (layer "B.Cu") (net 53))
+  (segment (start 84 73.5) (end 97.45 73.5) (width 0.6) (layer "B.Cu") (net 53))
+  (segment (start 110.5625 71.05) (end 108.05 71.05) (width 0.5) (layer "F.Cu") (net 55))
+  (segment (start 108.05 71.05) (end 106 69) (width 0.5) (layer "F.Cu") (net 55))
+  (via (at 106 69) (size 0.8) (drill 0.4) (layers "F.Cu" "B.Cu") (net 55))
+  (segment (start 106 69) (end 105.79 69) (width 0.5) (layer "B.Cu") (net 55))
+  (segment (start 105.79 69) (end 101.58 64.79) (width 0.5) (layer "B.Cu") (net 55))
   (zone (net 22) (net_name "GND") (layer "F.Cu") (hatch edge 0.508)
     (connect_pads (clearance 0.508))
